File: src/EDA/Circuits/Counter12Bits.kicad_pcb (KiCad board)
At the start: 2 copper layers, 144.8 x 44.4 mm, 29 parts, among them J1 Conn_01x03_Pin, J10 Conn_01x03_Pin, J11 Conn_01x03_Pin, J12 Conn_01x03_Pin, J13 Conn_01x03_Pin, J14 Conn_01x03_Pin, J15 Conn_01x03_Pin, J16 Conn_01x03_Pin, J17 Conn_01x04, J18 Conn_01x10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

Commit message: change pin lable from LOAD to LD
Other:
- board text added: "~{LD} 0-3"
- board text added: "~{LD} 4-7"
- board text added: "~{LD} 8-11"
- board text removed: "~{LOAD} 0-3"
- board text removed: "~{LOAD} 4-7"
- board text removed: "~{LOAD} 8-11"
Changed lines of the file:
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@@
 		)
 	)
-	(gr_text "~{LOAD}\n4-7"
+	(gr_text "~{LD}\n4-7"
 		(at 83.058 87.884 0)
 		(layer "F.SilkS")
@@
 		)
 	)
-	(gr_text "~{LOAD}\n8-11"
+	(gr_text "~{LD}\n8-11"
 		(at 110.998 87.884 0)
 		(layer "F.SilkS")
@@
 		)
 	)
-	(gr_text "~{LOAD}\n0-3"
+	(gr_text "~{LD}\n0-3"
 		(at 55.118 87.884 0)
 		(layer "F.SilkS")
